File: X13_Power_Distribution_D.sch (EAGLE design)
At the start: 44 parts, among them Q1 IRF1018EPBF, Q2 SSM3K341R, Q3 IRF1018EPBF, Q4 IRF1018EPBF, Q5 SSM3K341R, Q6 SSM3K341R, U1 LM74610, U2 LM74610, U3 LM5050, U4 LM5050

Commit message: Version D :/
Parts:
- removed BRICK_A, BRICK_B: DIST2BRICK_C, Brick_Dist_Connector:DIST2BRICK_C
- added BRICK1, BRICK2: DIST2BRICKVER_D2, Brick_Dist_Connector:DIST2BRICKVER_D2
Connections:
- net +12V_A: now also BRICK1.VOUT+; no longer BRICK_A.VOUT+
- net +12V_B: now also BRICK2.VOUT+; no longer BRICK_B.VOUT+
- net +48V: now also BRICK1.VIN+, BRICK2.VIN+; no longer BRICK_A.VIN+, BRICK_B.VIN+
- net 12V_GND: now also BRICK1.VOUT-, BRICK2.VOUT-; no longer BRICK_A.VOUT-, BRICK_B.VOUT-
- net 48V_GND: now also BRICK1.VIN-, BRICK2.VIN-; no longer BRICK_A.VIN-, BRICK_B.VIN-
- net ALERT_1: now also BRICK1.ALERT; no longer BRICK_A.ALERT
- net ALERT_2: now also BRICK2.ALERT; no longer BRICK_B.ALERT
- net C2_1: now also BRICK1.C2; no longer BRICK_A.C2
- net C2_2: now also BRICK2.C2; no longer BRICK_B.C2
- net CLK: now also BRICK1.CLK, BRICK2.CLK; no longer BRICK_A.CLK, BRICK_B.CLK
- net DATA: now also BRICK1.DATA, BRICK2.DATA; no longer BRICK_A.DATA, BRICK_B.DATA
- net ON/OFF: now also BRICK1.ON/OFF, BRICK2.ON/OFF; no longer BRICK_A.ON/OFF, BRICK_B.ON/OFF
Changed lines of the file:
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@@
 <part name="H4" library="Mounting Holes" deviceset="6-32-HOLE" device="" package3d_urn="urn:adsk.eagle:package:24384748/2"/>
 <part name="CONVERSION" library="Dist_Convert_Connector" deviceset="DIST2CON" device=""/>
-<part name="BRICK_A" library="Brick_Dist_Connector" deviceset="DIST2BRICK_C" device=""/>
-<part name="BRICK_B" library="Brick_Dist_Connector" deviceset="DIST2BRICK_C" device=""/>
 <part name="Q5" library="SparkFun-DiscreteSemi" library_urn="urn:adsk.eagle:library:514" deviceset="MOSFET-NCH" device="-2N7002PW" package3d_urn="urn:adsk.eagle:package:38456/1" value="SSM3K341R"/>
 <part name="D5" library="SparkFun-DiscreteSemi" library_urn="urn:adsk.eagle:library:514" deviceset="DIODE-ZENER" device="-BZT52C3V6S" package3d_urn="urn:adsk.eagle:package:38441/1" value="15V"/>
@@
 <part name="U3" library="Dist_OR_Controller" deviceset="DIST_OR_CONTROL_ALT" device="MK06A-M" value="LM5050"/>
 <part name="U4" library="Dist_OR_Controller" deviceset="DIST_OR_CONTROL_ALT" device="MK06A-M" value="LM5050"/>
+<part name="BRICK1" library="Brick_Dist_Connector" deviceset="DIST2BRICK" device="VER_D2"/>
+<part name="BRICK2" library="Brick_Dist_Connector" deviceset="DIST2BRICK" device="VER_D2"/>
 </parts>
 <sheets>
@@
 <attribute name="NAME" x="40.64" y="27.432" size="1.27" layer="95"/>
 </instance>
-<instance part="BRICK_A" gate="G$1" x="38.1" y="101.6" smashed="yes">
-<attribute name="NAME" x="38.608" y="110.236" size="1.778" layer="95"/>
-</instance>
-<instance part="BRICK_B" gate="G$1" x="38.1" y="63.5" smashed="yes">
-<attribute name="NAME" x="38.608" y="72.136" size="1.778" layer="95"/>
-</instance>
 <instance part="Q5" gate="NMOS" x="214.63" y="53.34" smashed="yes">
 <attribute name="NAME" x="213.36" y="57.15" size="1.778" layer="95" font="vector"/>
@@
 <attribute name="NAME" x="311.15" y="141.478" size="2.0828" layer="95" ratio="6" rot="SR0"/>
 <attribute name="VALUE" x="314.96" y="127" size="2.0828" layer="96" ratio="6" rot="SMR180"/>
+</instance>
+<instance part="BRICK1" gate="G$1" x="38.1" y="101.6" smashed="yes">
+<attribute name="NAME" x="38.608" y="110.236" size="1.778" layer="95"/>
+</instance>
+<instance part="BRICK2" gate="G$1" x="38.1" y="63.5" smashed="yes">
+<attribute name="NAME" x="38.608" y="72.136" size="1.778" layer="95"/>
 </instance>
 </instances>
@@
 <wire x1="68.58" y1="106.68" x2="72.39" y2="106.68" width="0.1524" layer="91"/>
 <label x="72.39" y="106.68" size="1.778" layer="95" xref="yes"/>
-<pinref part="BRICK_A" gate="G$1" pin="VOUT+"/>
+<pinref part="BRICK1" gate="G$1" pin="VOUT+"/>
 </segment>
 <segment>
@@
 <wire x1="68.58" y1="68.58" x2="72.39" y2="68.58" width="0.1524" layer="91"/>
 <label x="72.39" y="68.58" size="1.778" layer="95" xref="yes"/>
-<pinref part="BRICK_B" gate="G$1" pin="VOUT+"/>
+<pinref part="BRICK2" gate="G$1" pin="VOUT+"/>
 </segment>
 <segment>
@@
 <wire x1="33.02" y1="91.44" x2="29.21" y2="91.44" width="0.1524" layer="91"/>
 <label x="29.21" y="91.44" size="1.778" layer="95" rot="R180" xref="yes"/>
-<pinref part="BRICK_A" gate="G$1" pin="ON/OFF"/>
+<pinref part="BRICK1" gate="G$1" pin="ON/OFF"/>
 </segment>
 <segment>
 <wire x1="33.02" y1="53.34" x2="29.21" y2="53.34" width="0.1524" layer="91"/>
 <label x="29.21" y="53.34" size="1.778" layer="95" rot="R180" xref="yes"/>
-<pinref part="BRICK_B" gate="G$1" pin="ON/OFF"/>
+<pinref part="BRICK2" gate="G$1" pin="ON/OFF"/>
 </segment>
 </net>
@@
 <wire x1="33.02" y1="106.68" x2="29.21" y2="106.68" width="0.1524" layer="91"/>
 <label x="29.21" y="106.68" size="1.778" layer="95" rot="R180" xref="yes"/>
-<pinref part="BRICK_A" gate="G$1" pin="VIN+"/>
+<pinref part="BRICK1" gate="G$1" pin="VIN+"/>
 </segment>
 <segment>
 <wire x1="33.02" y1="68.58" x2="29.21" y2="68.58" width="0.1524" layer="91"/>
 <label x="29.21" y="68.58" size="1.778" layer="95" rot="R180" xref="yes"/>
-<pinref part="BRICK_B" gate="G$1" pin="VIN+"/>
+<pinref part="BRICK2" gate="G$1" pin="VIN+"/>
 </segment>
 <segment>
@@
 <wire x1="33.02" y1="101.6" x2="29.21" y2="101.6" width="0.1524" layer="91"/>
 <label x="29.21" y="101.6" size="1.778" layer="95" rot="R180" xref="yes"/>
-<pinref part="BRICK_A" gate="G$1" pin="VIN-"/>
+<pinref part="BRICK1" gate="G$1" pin="VIN-"/>
 </segment>
 <segment>
 <wire x1="33.02" y1="63.5" x2="29.21" y2="63.5" width="0.1524" layer="91"/>
 <label x="29.21" y="63.5" size="1.778" layer="95" rot="R180" xref="yes"/>
-<pinref part="BRICK_B" gate="G$1" pin="VIN-"/>
+<pinref part="BRICK2" gate="G$1" pin="VIN-"/>
 </segment>
 <segment>
@@
 <wire x1="68.58" y1="86.36" x2="72.39" y2="86.36" width="0.1524" layer="91"/>
 <label x="72.39" y="86.36" size="1.778" layer="95" xref="yes"/>
-<pinref part="BRICK_A" gate="G$1" pin="CLK"/>
+<pinref part="BRICK1" gate="G$1" pin="CLK"/>
 </segment>
 <segment>
 <wire x1="68.58" y1="48.26" x2="72.39" y2="48.26" width="0.1524" layer="91"/>
 <label x="72.39" y="48.26" size="1.778" layer="95" xref="yes"/>
-<pinref part="BRICK_B" gate="G$1" pin="CLK"/>
+<pinref part="BRICK2" gate="G$1" pin="CLK"/>
 </segment>
 </net>
@@
 <wire x1="68.58" y1="96.52" x2="72.39" y2="96.52" width="0.1524" layer="91"/>
 <label x="72.39" y="96.52" size="1.778" layer="95" xref="yes"/>
-<pinref part="BRICK_A" gate="G$1" pin="DATA"/>
+<pinref part="BRICK1" gate="G$1" pin="DATA"/>
 </segment>
 <segment>
 <wire x1="68.58" y1="58.42" x2="72.39" y2="58.42" width="0.1524" layer="91"/>
 <label x="72.39" y="58.42" size="1.778" layer="95" xref="yes"/>
-<pinref part="BRICK_B" gate="G$1" pin="DATA"/>
+<pinref part="BRICK2" gate="G$1" pin="DATA"/>
 </segment>
 </net>
@@
 <wire x1="68.58" y1="101.6" x2="72.39" y2="101.6" width="0.1524" layer="91"/>
 <label x="72.39" y="101.6" size="1.778" layer="95" xref="yes"/>
-<pinref part="BRICK_A" gate="G$1" pin="VOUT-"/>
+<pinref part="BRICK1" gate="G$1" pin="VOUT-"/>
 </segment>
 <segment>
 <wire x1="68.58" y1="63.5" x2="72.39" y2="63.5" width="0.1524" layer="91"/>
 <label x="72.39" y="63.5" size="1.778" layer="95" xref="yes"/>
-<pinref part="BRICK_B" gate="G$1" pin="VOUT-"/>
+<pinref part="BRICK2" gate="G$1" pin="VOUT-"/>
 </segment>
 <segment>
@@
 <wire x1="68.58" y1="43.18" x2="72.39" y2="43.18" width="0.1524" layer="91"/>
 <label x="72.39" y="43.18" size="1.778" layer="95" xref="yes"/>
-<pinref part="BRICK_B" gate="G$1" pin="C2"/>
+<pinref part="BRICK2" gate="G$1" pin="C2"/>
 </segment>
 </net>
@@
 <wire x1="68.58" y1="81.28" x2="72.39" y2="81.28" width="0.1524" layer="91"/>
 <label x="72.39" y="81.28" size="1.778" layer="95" xref="yes"/>
-<pinref part="BRICK_A" gate="G$1" pin="C2"/>
+<pinref part="BRICK1" gate="G$1" pin="C2"/>
 </segment>
 </net>
@@
 <wire x1="68.58" y1="53.34" x2="72.39" y2="53.34" width="0.1524" layer="91"/>
 <label x="72.39" y="53.34" size="1.778" layer="95" xref="yes"/>
-<pinref part="BRICK_B" gate="G$1" pin="ALERT"/>
+<pinref part="BRICK2" gate="G$1" pin="ALERT"/>
 </segment>
 </net>
@@
 <wire x1="68.58" y1="91.44" x2="72.39" y2="91.44" width="0.1524" layer="91"/>
 <label x="72.39" y="91.44" size="1.778" layer="95" xref="yes"/>
-<pinref part="BRICK_A" gate="G$1" pin="ALERT"/>
-</segment>
-</net>
+<pinref part="BRICK1" gate="G$1" pin="ALERT"/>
+</segment>
+</net>
