File: X13_Power_Distribution_D.brd (EAGLE design)
At the start: 152.4 x 73.7 mm, 44 parts, among them Q1 IRF1018EPBF, Q2 SSM3K341R, Q3 IRF1018EPBF, Q4 IRF1018EPBF, Q5 SSM3K341R, Q6 SSM3K341R, U1 LM74610, U2 LM74610, U3 LM5050, U4 LM5050

Commit message: Version D :/
Parts:
- removed BRICK_A, BRICK_B: DIST2BRICK_C, Brick_Dist_Connector:DIST2BRICK_C
- added BRICK1, BRICK2: DIST2BRICKVER_D2, Brick_Dist_Connector:DIST2BRICK_D2
- moved BACKPLANE_LOGIC 92.8 mm to (118.1, 7.62)
- moved C3 78.8 mm to (-8.89, 15.2)
- moved R5 64.6 mm to (128.3, 19.1), turned to 0 degrees
- moved R4 46.2 mm to (128.3, 16.5)
- moved R6 45.6 mm to (128.3, 21.6)
- moved R7 45.6 mm to (128.3, 24.1)
- moved D8 21.7 mm to (110.5, 21.6), turned to 0 degrees
- moved D7 20.7 mm to (118.1, 34.3)
- moved D1 20.7 mm to (82.5, 69.8), turned to 180 degrees
- moved R11 20.5 mm to (115.6, 21.6), turned to 0 degrees
- moved Q6 17.8 mm to (120.7, 27.9)
- moved R10 16.7 mm to (120.7, 31.8)
- moved 5V_POE 16.5 mm to (127.0, -6.35)
- moved BACKPLANE_PWR 12.7 mm to (76.2, 0.00)
- moved U4 12.5 mm to (115.6, 27.9), turned to 180 degrees
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Connections:
- net +12V_A: now also BRICK1.2@1, BRICK1.2@10, BRICK1.2@11, BRICK1.2@12, BRICK1.2@13, BRICK1.2@14, BRICK1.2@15, BRICK1.2@16, BRICK1.2@17, BRICK1.2@18, BRICK1.2@19, BRICK1.2@2, BRICK1.2@20, BRICK1.2@3, BRICK1.2@4, BRICK1.2@5, BRICK1.2@6, BRICK1.2@7, BRICK1.2@8, BRICK1.2@9; no longer BRICK_A.2@1, BRICK_A.2@10, BRICK_A.2@11, BRICK_A.2@12, BRICK_A.2@13, BRICK_A.2@14, BRICK_A.2@15, BRICK_A.2@16, BRICK_A.2@2, BRICK_A.2@3, BRICK_A.2@4, BRICK_A.2@5, BRICK_A.2@6, BRICK_A.2@7, BRICK_A.2@8, BRICK_A.2@9
- net +12V_B: now also BRICK2.2@1, BRICK2.2@10, BRICK2.2@11, BRICK2.2@12, BRICK2.2@13, BRICK2.2@14, BRICK2.2@15, BRICK2.2@16, BRICK2.2@17, BRICK2.2@18, BRICK2.2@19, BRICK2.2@2, BRICK2.2@20, BRICK2.2@3, BRICK2.2@4, BRICK2.2@5, BRICK2.2@6, BRICK2.2@7, BRICK2.2@8, BRICK2.2@9; no longer BRICK_B.2@1, BRICK_B.2@10, BRICK_B.2@11, BRICK_B.2@12, BRICK_B.2@13, BRICK_B.2@14, BRICK_B.2@15, BRICK_B.2@16, BRICK_B.2@2, BRICK_B.2@3, BRICK_B.2@4, BRICK_B.2@5, BRICK_B.2@6, BRICK_B.2@7, BRICK_B.2@8, BRICK_B.2@9
- net +48V: now also BRICK1.1@1, BRICK1.1@10, BRICK1.1@2, BRICK1.1@3, BRICK1.1@4, BRICK1.1@5, BRICK1.1@6, BRICK1.1@7, BRICK1.1@8, BRICK1.1@9, BRICK2.1@1, BRICK2.1@10, BRICK2.1@2, BRICK2.1@3, BRICK2.1@4, BRICK2.1@5, BRICK2.1@6, BRICK2.1@7, BRICK2.1@8, BRICK2.1@9; no longer BRICK_A.1@1, BRICK_A.1@10, BRICK_A.1@2, BRICK_A.1@3, BRICK_A.1@4, BRICK_A.1@5, BRICK_A.1@6, BRICK_A.1@7, BRICK_A.1@8, BRICK_A.1@9, BRICK_B.1@1, BRICK_B.1@10, BRICK_B.1@2, BRICK_B.1@3, BRICK_B.1@4, BRICK_B.1@5, BRICK_B.1@6, BRICK_B.1@7, BRICK_B.1@8, BRICK_B.1@9
- net 12V_GND: now also BRICK1.4@1, BRICK1.4@10, BRICK1.4@11, BRICK1.4@12, BRICK1.4@13, BRICK1.4@14, BRICK1.4@15, BRICK1.4@16, BRICK1.4@17, BRICK1.4@18, BRICK1.4@19, BRICK1.4@2, BRICK1.4@20, BRICK1.4@3, BRICK1.4@4, BRICK1.4@5, BRICK1.4@6, BRICK1.4@7, BRICK1.4@8, BRICK1.4@9, BRICK2.4@1, BRICK2.4@10, BRICK2.4@11, BRICK2.4@12, BRICK2.4@13, BRICK2.4@14, BRICK2.4@15, BRICK2.4@16, BRICK2.4@17, BRICK2.4@18, BRICK2.4@19, BRICK2.4@2, BRICK2.4@20, BRICK2.4@3, BRICK2.4@4, BRICK2.4@5, BRICK2.4@6, BRICK2.4@7, BRICK2.4@8, BRICK2.4@9; no longer BRICK_A.4@1, BRICK_A.4@10, BRICK_A.4@11, BRICK_A.4@12, BRICK_A.4@13, BRICK_A.4@14, BRICK_A.4@15, BRICK_A.4@16, BRICK_A.4@2, BRICK_A.4@3, BRICK_A.4@4, BRICK_A.4@5, BRICK_A.4@6, BRICK_A.4@7, BRICK_A.4@8, BRICK_A.4@9, BRICK_B.4@1, BRICK_B.4@10, BRICK_B.4@11, BRICK_B.4@12, BRICK_B.4@13, BRICK_B.4@14, BRICK_B.4@15, BRICK_B.4@16, BRICK_B.4@2, BRICK_B.4@3, BRICK_B.4@4, BRICK_B.4@5, BRICK_B.4@6, BRICK_B.4@7, BRICK_B.4@8, BRICK_B.4@9
- net 48V_GND: now also BRICK1.3@1, BRICK1.3@10, BRICK1.3@2, BRICK1.3@3, BRICK1.3@4, BRICK1.3@5, BRICK1.3@6, BRICK1.3@7, BRICK1.3@8, BRICK1.3@9, BRICK2.3@1, BRICK2.3@10, BRICK2.3@2, BRICK2.3@3, BRICK2.3@4, BRICK2.3@5, BRICK2.3@6, BRICK2.3@7, BRICK2.3@8, BRICK2.3@9; no longer BRICK_A.3@1, BRICK_A.3@10, BRICK_A.3@2, BRICK_A.3@3, BRICK_A.3@4, BRICK_A.3@5, BRICK_A.3@6, BRICK_A.3@7, BRICK_A.3@8, BRICK_A.3@9, BRICK_B.3@1, BRICK_B.3@10, BRICK_B.3@2, BRICK_B.3@3, BRICK_B.3@4, BRICK_B.3@5, BRICK_B.3@6, BRICK_B.3@7, BRICK_B.3@8, BRICK_B.3@9
- net ALERT_1: now also BRICK1.D; no longer BRICK_A.D
- net ALERT_2: now also BRICK2.D; no longer BRICK_B.D
- net C2_1: now also BRICK1.A; no longer BRICK_A.A
- net C2_2: now also BRICK2.A; no longer BRICK_B.A
- net CLK: now also BRICK1.C, BRICK2.C; no longer BRICK_A.C, BRICK_B.C
- net DATA: now also BRICK1.E, BRICK2.E; no longer BRICK_A.E, BRICK_B.E
- net ON/OFF: now also BRICK1.B, BRICK2.B; no longer BRICK_A.B, BRICK_B.B
Routing:
- net +3.3V: track 207.5 -> 42.0 mm, vias 5 -> 1
- net +5V: track 153.0 -> 31.6 mm, vias 2 -> 0
- net 5V_GND: track 120.4 -> 22.2 mm, vias 2 -> 0
- net +12V: track 111.2 -> 46.4 mm, vias 6 -> 2
- net C2_1: track 72.0 -> 123.9 mm, vias 1 -> 0
- net DATA: track 79.3 -> 123.9 mm
- net CLK: track 77.9 -> 121.3 mm
- net OR_DRIVE_A: track 43.4 -> 0.00 mm
- net ALERT_1: track 74.2 -> 117.4 mm, vias 3 -> 2
- net ALERT_2: track 66.3 -> 107.6 mm, vias 4 -> 1
- net 12V_GND: track 60.8 -> 19.9 mm, vias 12 -> 1
- net REV_DRIVE: track 28.9 -> 0.00 mm, vias 1 -> 0
- net +12V_A: track 25.4 -> 0.00 mm, vias 3 -> 0
- net OR_DRIVE_B: track 48.4 -> 32.6 mm, vias 4 -> 2
- net N$1: track 15.2 -> 0.00 mm, vias 1 -> 0
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- removed copper zone on layer 1, net +12V_A
- removed copper zone on layer 1, net +12V_B
- removed copper zone on layer 1, net 12V_GND
Other:
- outline, holes or cut-outs redrawn

Commit message: Uses brick connector vD2
Parts:
- moved C3 85.2 mm to (71.1, 44.5)
- moved U3 30.9 mm to (48.3, 38.1)
- moved 5V_POE 20.8 mm to (110.5, 6.35), turned to 0 degrees
- moved C1 20.5 mm to (55.9, 40.6)
- moved D5 19.2 mm to (40.6, 35.6), turned to 90 degrees
- moved U1 19.1 mm to (55.9, 36.8)
- moved R8 16.9 mm to (38.1, 40.6), turned to 270 degrees
- moved Q5 14.9 mm to (36.8, 36.8), turned to 180 degrees
- moved D6 14.5 mm to (43.2, 36.8)
- moved Q3 14.0 mm to (50.8, 27.9)
- moved R9 12.7 mm to (36.8, 33.0)
Routing:
- net +12V: track 46.4 -> 98.1 mm, vias 2 -> 5
- net 5V_GND: track 22.2 -> 47.6 mm, vias 0 -> 1
- net OR_DRIVE_A: track 0.00 -> 24.4 mm
- net 12V_GND: track 19.9 -> 43.5 mm, vias 1 -> 7
- net +12V_A: track 0.00 -> 18.2 mm, vias 0 -> 1
- net N$1: track 0.00 -> 15.3 mm, vias 0 -> 1
- net N$5: track 0.00 -> 11.6 mm, vias 0 -> 2
- net +5V: track 31.6 -> 43.1 mm, vias 0 -> 1
- net ON/OFF: track 63.2 -> 73.8 mm, vias 0 -> 1
- net VCAPH_A: track 0.00 -> 9.17 mm
- net ON/OFF_DRIVE: track 0.00 -> 8.10 mm
- net +12V_B: track 15.0 -> 22.9 mm, vias 0 -> 2
- net VCAPL_A: track 0.00 -> 6.36 mm
- net LED_DRIVE_A: track 0.00 -> 5.52 mm
- net C2_1: track 123.9 -> 121.5 mm
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- added copper zone on layer 1, net +12V_A
- added copper zone on layer 1, net 12V_GND
- added copper zone on layer 1, net N$2
Other:
- board text added: "5V_GND"
- board text removed: "5V_ETHERNET"
