File: X13_Power_Distribution_D1.brd (EAGLE design)
At the start: 152.4 x 73.7 mm, 44 parts, among them Q1 IRF1018EPBF, Q2 SSM3K341R, Q3 IRF1018EPBF, Q4 IRF1018EPBF, Q5 SSM3K341R, Q6 SSM3K341R, U1 LM74610, U2 LM74610, U3 LM5050, U4 LM5050

Commit message: Tweaks
Parts:
- moved R1 29.2 mm to (83.8, 59.7), turned to 0 degrees
- moved 5V_POE 21.6 mm to (132.1, 7.62)
- moved BACKPLANE_PWR 11.0 mm to (65.2, 0.00)
- moved BACKPLANE_LOGIC 10.2 mm to (108.0, 7.62)
- moved Q1 8.98 mm to (69.8, 58.4)
- moved D1 7.73 mm to (83.8, 62.2)
- moved TETHER 6.35 mm to (26.7, 58.4)
- moved 48V_POE 2.84 mm to (14.0, 67.3), turned to 0 degrees
Routing:
- net DATA: track 125.6 -> 99.4 mm
- net C2_2: track 96.1 -> 114.9 mm
- net 5V_GND: track 47.6 -> 32.4 mm
- net ALERT_1: track 118.0 -> 103.0 mm
- net +3.3V: track 42.0 -> 54.2 mm, vias 1 -> 2
- net C2_1: track 121.5 -> 130.7 mm
- net REV_DRIVE: track 0.00 -> 8.96 mm, vias 0 -> 1
- net ALERT_2: track 108.6 -> 101.7 mm
- net +5V: track 43.1 -> 40.0 mm
- net CLK: track 120.8 -> 122.1 mm
- added copper zone on layer 1, net +5V
- added copper zone on layer 1, net 5V_GND

Commit message: V1
Parts:
- moved D2 10.1 mm to (109.2, 53.1), turned to 180 degrees
- moved R3 5.39 mm to (113.8, 54.4), turned to 0 degrees
- moved R2 4.58 mm to (96.5, 54.6)
- moved D4 3.81 mm to (109.2, 55.9), turned to 180 degrees
- moved Q2 3.59 mm to (104.6, 56.1)
- moved D3 1.52 mm to (102.9, 53.1)
Routing:
- net 5V_GND: track 32.4 -> 63.3 mm, vias 1 -> 2
- net N$1: track 15.3 -> 4.05 mm
- net ON/OFF: track 73.8 -> 66.1 mm
- net N$4: track 0.00 -> 2.04 mm
- net ON/OFF_DRIVE: track 8.10 -> 10.0 mm
- net C2_2: track 114.9 -> 113.1 mm
- net +3.3V: track 54.2 -> 55.8 mm
- net C2_1: track 130.7 -> 129.1 mm
- net +12V_A: track 16.4 -> 18.0 mm, vias 2 -> 1
- net CLK: track 122.1 -> 120.7 mm
- net ALERT_2: track 101.7 -> 100.6 mm
- net ALERT_1: track 103.0 -> 102.1 mm
- net DATA: track 99.4 -> 98.7 mm
- net 12V_GND: track 43.5 -> 43.6 mm, vias 7 -> 8
- net +5V: vias 1 -> 0
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- added copper zone on layer 1, net +12V_B
- removed copper zone on layer 1, net N$2
Other:
- board text added: "ROV X13 Distribution v1 Sam Kovnar Read Hedl Grant Geyer January 9, 2021"
- board text removed: "+5V"
- board text removed: "5V_GND"
