File: X13_Power_Distribution.brd (EAGLE design)
At the start: 152.4 x 73.7 mm, 52 parts, among them Q1 IRF1018EPBF, Q2 SSM3K341R, Q3 IRF1018EPBF, Q4 IRF1018EPBF, Q5 SSM3K341R, Q6 SSM3K341R, Q7 SSM3K341R, Q8 SSM3K341R, U3 LM5050, U4 LM5050

Commit message: Add diode to on/off to discharge gate when power supply hits 0
Parts:
- added D10: 250mA/100V, SparkFun-DiscreteSemi:SOD-323
- added J1: (no value), SparkFun-Connectors:1X02
- added J2: (no value), SparkFun-Connectors:1X01
- +12V_A_TEST, +12V_B_TEST, +12V_TEST, +48V_TEST, 12_GND, 48GND_TEST: value SSW-101-02-G-S -> (none); device con-samtec:SSW-101-02-G-S -> SparkFun-Connectors:1X01
- moved +12V_TEST 0.92 mm to (82.0, 22.9)
- moved D9 0.51 mm to (99.6, 53.6)
Connections:
- net +48V: now also D10.C
- net CLK: now also J1.1
- net DATA: now also J1.2
- net ON/OFF: now also J2.1
- net ON/OFF_DRIVE: now also D10.A
Routing:
- net +12V: track 84.0 -> 62.7 mm, vias 2 -> 0
- net DATA: track 98.7 -> 112.4 mm, vias 1 -> 2
- net CLK: track 120.7 -> 126.9 mm, vias 1 -> 2
- net +48V: track 30.8 -> 34.3 mm
- net ON/OFF: track 63.4 -> 64.9 mm
- net ON/OFF_DRIVE: track 1.53 -> 2.98 mm, vias 0 -> 1
- net +12V_A: vias 0 -> 7
- added copper zone on layer 16, net +12V_A
- added copper zone on layer 1, net X
Other:
- board text added: "CLK - DATA"
- board text added: "On/Off"
